Commit message: update path to ros2 format

File: turtlebot3_gazebo/urdf/turtlebot3_burger.urdf (robot description, URDF)
Before this commit: robot turtlebot3_burger, 7 links, 6 joints
Links:
- link base_link: geometry collision box size=0.140 0.140 0.143; visual mesh filename=$(find turtlebot3_gazebo)/models/turtlebot3_common/meshes/b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 scale=0.001 0.001 0.001
- link base_scan: geometry collision cylinder length=0.0315 radius=0.055; visual mesh filename=$(find turtlebot3_gazebo)/models/turtlebot3_common/meshes/l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 scale=0.001 0.001 0.001
- link wheel_left_link: geometry collision cylinder length=0.018 radius=0.033; visual mesh filename=$(find turtlebot3_gazebo)/models/turtlebot3_common/meshes/t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 scale=0.001 0.001 0.001
- link wheel_right_link: geometry collision cylinder length=0.018 radius=0.033; visual mesh filename=$(find turtlebot3_gazebo)/models/turtlebot3_common/meshes/t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 scale=0.001 0.001 0.001

File: turtlebot3_gazebo/urdf/turtlebot3_waffle.urdf (robot description, URDF)
Before this commit: robot turtlebot3_waffle, 13 links, 12 joints
Links:
- link base_link: geometry collision box size=0.266 0.266 0.094; visual mesh filename=$(find turtlebot3_gazebo)/models/turtlebot3_common/meshes/w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 scale=0.001 0.001 0.001
- link base_scan: geometry collision cylinder length=0.0315 radius=0.055; visual mesh filename=$(find turtlebot3_gazebo)/models/turtlebot3_common/meshes/l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 scale=0.001 0.001 0.001
- link camera_link: geometry collision box size=0.012 0.132 0.020; visual mesh filename=$(find turtlebot3_gazebo)/models/turtlebot3_common/meshes/r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
- link wheel_left_link: geometry collision cylinder length=0.018 radius=0.033; visual mesh filename=$(find turtlebot3_gazebo)/models/turtlebot3_common/meshes/t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 scale=0.001 0.001 0.001
- link wheel_right_link: geometry collision cylinder length=0.018 radius=0.033; visual mesh filename=$(find turtlebot3_gazebo)/models/turtlebot3_common/meshes/t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 scale=0.001 0.001 0.001

File: turtlebot3_gazebo/urdf/turtlebot3_waffle_pi.urdf (robot description, URDF)
Before this commit: robot turtlebot3_waffle_pi, 11 links, 10 joints
Links:
- link base_link: geometry collision box size=0.266 0.266 0.094; visual mesh filename=$(find turtlebot3_gazebo)/models/turtlebot3_common/meshes/w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 scale=0.001 0.001 0.001
- link base_scan: geometry collision cylinder length=0.0315 radius=0.055; visual mesh filename=$(find turtlebot3_gazebo)/models/turtlebot3_common/meshes/l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 scale=0.001 0.001 0.001
- link wheel_left_link: geometry collision cylinder length=0.018 radius=0.033; visual mesh filename=$(find turtlebot3_gazebo)/models/turtlebot3_common/meshes/t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 scale=0.001 0.001 0.001
- link wheel_right_link: geometry collision cylinder length=0.018 radius=0.033; visual mesh filename=$(find turtlebot3_gazebo)/models/turtlebot3_common/meshes/t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 scale=0.001 0.001 0.001

Commit message: update path to original

File: turtlebot3_gazebo/urdf/turtlebot3_burger.urdf (robot description, URDF)
Before this commit: robot turtlebot3_burger, 7 links, 6 joints
Links:
- link base_link: geometry collision box size=0.140 0.140 0.143; visual mesh filename=package://turtlebot3_gazebo/models/turtlebot3_common/meshes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 scale=0.001 0.001 0.001
- link base_scan: geometry collision cylinder length=0.0315 radius=0.055; visual mesh filename=package://turtlebot3_gazebo/models/turtlebot3_common/meshes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 scale=0.001 0.001 0.001
- link wheel_left_link: geometry collision cylinder length=0.018 radius=0.033; visual mesh filename=package://turtlebot3_gazebo/models/turtlebot3_common/meshes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 scale=0.001 0.001 0.001
- link wheel_right_link: geometry collision cylinder length=0.018 radius=0.033; visual mesh filename=package://turtlebot3_gazebo/models/turtlebot3_common/meshes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 scale=0.001 0.001 0.001
